File: Kicad-Faraday/$GPS.sch (KiCad schematic (older format))
At the start: 5 parts, among them U7 M10478-A2

Commit message: Saving current RevD, need ot export BOM
Parts:
- gave numbers to parts that had none: 1
Changed lines of the file:
@@
 	4400 5050 7300 5050
 $Comp
-L C C?
+L C C15
 U 1 1 582878DD
 P 6800 4550
-F 0 "C?" V 6850 4600 50  0000 L CNN
+F 0 "C15" V 6850 4600 50  0000 L CNN
 F 1 "12pF" V 6850 4300 50  0000 L CNN
 F 2 "C0402" V 6750 4750 50  0000 C CNN
