File: Kicad-Faraday/RF_Front_End.sch (KiCad schematic (older format))
At the start: 18 parts, among them U4 CC1190, U5 SF2049E

Commit message: Saving current RevD, need ot export BOM
Parts:
- C32, C36: value 0.01uF -> 0.1uF
Changed lines of the file:
@@
 P 9400 3100
 F 0 "C32" V 9450 3175 50  0000 L CNN
-F 1 "0.01uF" V 9450 2775 50  0000 L CNN
+F 1 "0.1uF" V 9450 2775 50  0000 L CNN
 F 2 "C0402" V 9350 2900 50  0000 C CNN
 F 3 "" H 9400 3100 60  0000 C CNN
@@
 P 8200 4100
 F 0 "C36" V 8250 3900 50  0000 L CNN
-F 1 "0.01uF" V 8250 4150 50  0000 L CNN
+F 1 "0.1uF" V 8250 4150 50  0000 L CNN
 F 2 "C0402" V 8150 3925 50  0000 C CNN
 F 3 "" H 8200 4100 60  0000 C CNN

Commit message: Updated notes for PDF schematic. Check PSU routing and seems OK
Other:
- note added: "915MHz SAW Filter"
- note removed: "900MHz SAW Filter"
Changed lines of the file:
@@
 $EndComp
 Text Notes 12100 5300 0    60   ~ 12
-900MHz SAW Filter
+915MHz SAW Filter
 $Comp
 L +3.3V #PWR061
@@
 	1    0    0    -1
 $EndComp
-Text Notes 13100 5100 0    120  ~ 24
+Text Notes 14500 5800 0    120  ~ 24
 Input
-Text Notes 2750 5300 0    120  ~ 24
+Text Notes 1650 5550 0    120  ~ 24
 Output
 Text Label 7100 5500 0    60   ~ 0
